Commit message: Add camera_link to urdf
In order to simulate the camera there must be a camera_link in the tf
tree to relate the camera coordinate frame to the base robot frame.
The link is currently floating but is in a position which is relatively
close to where it will be mounted.

File: ros_ws/src/robot_description/robots/igvc.urdf.xacro (robot description, xacro)
@@ -168,4 +168,27 @@
             <axis xyz="0 0 0" />
         </joint>
+        <link name="camera_link">
+            <visual>
+                <origin xyz="0 0 0" rpy="0 0 0" />
+                <geometry>
+                    <box size=".03 .05 .05"/>
+                </geometry>
+                <material name="">
+                    <color rgba="0 0 0 .7" />
+                </material>
+            </visual>
+            <collision>
+                <origin xyz="0 0 0" rpy="0 0 0" />
+                <geometry>
+                    <box size=".03 .05 .05"/>
+                </geometry>
+            </collision>
+        </link>
+        <joint name="camera_joint" type="fixed">
+            <origin xyz="-0.20 0.34722 .6" rpy="0 0.5235 0"/>
+            <parent link="base_link"/>
+            <child link="camera_link"/>
+            <axis xyz="0 0 0" />
+        </joint>
         <igvc_sim/>
     </xacro:macro>
